Commit message: Remove ros_control references from URDF

File: leo_description/urdf/macros.xacro (robot description, xacro)
@@ -303,65 +303,4 @@
       </plugin>
     </gazebo>
-    <!-- ros_control plugin -->
-    <gazebo>
-      <plugin name="gazebo_ros_control" filename="libgazebo_ros_control.so">
-        <robotNamespace>${robot_ns}</robotNamespace>
-        <robotSimType>gazebo_ros_control/DefaultRobotHWSim</robotSimType>
-      </plugin>
-    </gazebo>
-    <transmission name="wheel_FL_trans">
-      <type>transmission_interface/SimpleTransmission</type>
-      <joint name="wheel_FL_joint">
-        <hardwareInterface>hardware_interface/VelocityJointInterface</hardwareInterface>
-      </joint>
-      <actuator name="wheel_FL_motor">
-        <mechanicalReduction>1</mechanicalReduction>
-        <hardwareInterface>hardware_interface/VelocityJointInterface</hardwareInterface>
-      </actuator>
-    </transmission>
-    <transmission name="wheel_RL_trans">
-      <type>transmission_interface/SimpleTransmission</type>
-      <joint name="wheel_RL_joint">
-        <hardwareInterface>hardware_interface/VelocityJointInterface</hardwareInterface>
-      </joint>
-      <actuator name="wheel_RL_motor">
-        <mechanicalReduction>1</mechanicalReduction>
-        <hardwareInterface>hardware_interface/VelocityJointInterface</hardwareInterface>
-      </actuator>
-    </transmission>
-    <transmission name="wheel_FR_trans">
-      <type>transmission_interface/SimpleTransmission</type>
-      <joint name="wheel_FR_joint">
-        <hardwareInterface>hardware_interface/VelocityJointInterface</hardwareInterface>
-      </joint>
-      <actuator name="wheel_FR_motor">
-        <mechanicalReduction>1</mechanicalReduction>
-        <hardwareInterface>hardware_interface/VelocityJointInterface</hardwareInterface>
-      </actuator>
-    </transmission>
-    <transmission name="wheel_RR_trans">
-      <type>transmission_interface/SimpleTransmission</type>
-      <joint name="wheel_RR_joint">
-        <hardwareInterface>hardware_interface/VelocityJointInterface</hardwareInterface>
-      </joint>
-      <actuator name="wheel_RR_motor">
-        <mechanicalReduction>1</mechanicalReduction>
-        <hardwareInterface>hardware_interface/VelocityJointInterface</hardwareInterface>
-      </actuator>
-    </transmission>
-    <transmission name="rocker_L_trans">
-      <type>transmission_interface/SimpleTransmission</type>
-      <joint name="rocker_L_joint">
-        <hardwareInterface>hardware_interface/EffortJointInterface</hardwareInterface>
-      </joint>
-      <actuator name="rocker_L_virtual_motor"/>
-    </transmission>
-    <transmission name="rocker_R_trans">
-      <type>transmission_interface/SimpleTransmission</type>
-      <joint name="rocker_R_joint">
-        <hardwareInterface>hardware_interface/EffortJointInterface</hardwareInterface>
-      </joint>
-      <actuator name="rocker_R_virtual_motor"/>
-    </transmission>
   </xacro:macro>
   <xacro:macro name="leo_sim"

Commit message: Initial gazebo_ros2_control configuration

File: leo_description/urdf/macros.xacro (robot description, xacro)
@@ -295,14 +295,56 @@
       </plugin>
     </gazebo>
-    <!-- joint state publisher -->
+    <ros2_control name="GazeboSystem" type="system">
+      <hardware>
+        <plugin>gazebo_ros2_control/GazeboSystem</plugin>
+      </hardware>
+      <joint name="rocker_L_joint">
+        <state_interface name="position"/>
+      </joint>
+      <joint name="rocker_R_joint">
+        <state_interface name="position"/>
+      </joint>
+      <joint name="wheel_FL_joint">
+        <command_interface name="effort">
+          <param name="min">-1000</param>
+          <param name="max">1000</param>
+        </command_interface>
+        <state_interface name="position"/>
+        <state_interface name="velocity"/>
+        <state_interface name="effort"/>
+      </joint>
+      <joint name="wheel_RL_joint">
+        <command_interface name="effort">
+          <param name="min">-1000</param>
+          <param name="max">1000</param>
+        </command_interface>
+        <state_interface name="position"/>
+        <state_interface name="velocity"/>
+        <state_interface name="effort"/>
+      </joint>
+      <joint name="wheel_FR_joint">
+        <command_interface name="effort">
+          <param name="min">-1000</param>
+          <param name="max">1000</param>
+        </command_interface>
+        <state_interface name="position"/>
+        <state_interface name="velocity"/>
+        <state_interface name="effort"/>
+      </joint>
+      <joint name="wheel_RR_joint">
+        <command_interface name="effort">
+          <param name="min">-1000</param>
+          <param name="max">1000</param>
+        </command_interface>
+        <state_interface name="position"/>
+        <state_interface name="velocity"/>
+        <state_interface name="effort"/>
+      </joint>
+    </ros2_control>
     <gazebo>
-      <plugin name="joint_state_publisher" filename="libgazebo_ros_joint_state_publisher.so">
-        <update_rate>20</update_rate>
-        <joint_name>rocker_L_joint</joint_name>
-        <joint_name>rocker_R_joint</joint_name>
-        <joint_name>wheel_FL_joint</joint_name>
-        <joint_name>wheel_RL_joint</joint_name>
-        <joint_name>wheel_FR_joint</joint_name>
-        <joint_name>wheel_RR_joint</joint_name>
+      <plugin filename="libgazebo_ros2_control.so" name="gazebo_ros2_control">
+        <robot_param>robot_description</robot_param>
+        <robot_param_node>robot_state_publisher</robot_param_node>
+        <parameters>package://leo_description/config/controllers.yaml</parameters>
       </plugin>
     </gazebo>

Commit message: Add diff_drive_controller

File: leo_description/urdf/macros.xacro (robot description, xacro)
@@ -306,7 +306,7 @@
       </joint>
       <joint name="wheel_FL_joint">
-        <command_interface name="effort">
-          <param name="min">-1000</param>
-          <param name="max">1000</param>
+        <command_interface name="velocity">
+          <param name="min">-6</param>
+          <param name="max">6</param>
         </command_interface>
         <state_interface name="position"/>
@@ -315,7 +315,7 @@
       </joint>
       <joint name="wheel_RL_joint">
-        <command_interface name="effort">
-          <param name="min">-1000</param>
-          <param name="max">1000</param>
+        <command_interface name="velocity">
+          <param name="min">-6</param>
+          <param name="max">6</param>
         </command_interface>
         <state_interface name="position"/>
@@ -324,7 +324,7 @@
       </joint>
       <joint name="wheel_FR_joint">
-        <command_interface name="effort">
-          <param name="min">-1000</param>
-          <param name="max">1000</param>
+        <command_interface name="velocity">
+          <param name="min">-6</param>
+          <param name="max">6</param>
         </command_interface>
         <state_interface name="position"/>
@@ -333,7 +333,7 @@
       </joint>
       <joint name="wheel_RR_joint">
-        <command_interface name="effort">
-          <param name="min">-1000</param>
-          <param name="max">1000</param>
+        <command_interface name="velocity">
+          <param name="min">-6</param>
+          <param name="max">6</param>
         </command_interface>
         <state_interface name="position"/>
@@ -367,5 +367,5 @@
         <parent link="world"/>
         <child link="${link_prefix}base_footprint"/>
-        <origin xyz="0.0 0.0 0"/>
+        <origin xyz="0.0 0.0 1.0"/>
       </joint>
     </xacro:if>

Commit message: Import changes from ROS1 port

File: leo_description/urdf/macros.xacro (robot description, xacro)
@@ -6,5 +6,6 @@
                        footprint_link:=true
                        link_prefix:=''
-                       joint_prefix:=''">
+                       joint_prefix:=''
+                       imu_translation:='0.0628 -0.0314 -0.0393'">
     <xacro:macro name="rocker_link" params="name">
       <link name="${link_prefix}rocker_${name}_link">
@@ -118,4 +119,5 @@
     <link name="${link_prefix}camera_frame"/>
     <link name="${link_prefix}camera_optical_frame"/>
+    <link name="${link_prefix}imu_frame"/>
     <!-- JOINTS -->
     <xacro:if value="${footprint_link}">
@@ -198,4 +200,9 @@
       <child link="${link_prefix}camera_optical_frame"/>
     </joint>
+    <joint name="${joint_prefix}imu_joint" type="fixed">
+      <origin xyz="${imu_translation}" rpy="0 0 0"/>
+      <parent link="${link_prefix}base_link"/>
+      <child link="${link_prefix}imu_frame"/>
+    </joint>
   </xacro:macro>
   <!-- LEO GAZEBO -->
@@ -206,8 +213,25 @@
       <xacro:property name="link_prefix" value="${robot_ns}/"/>
     </xacro:if>
+    <!-- base ODE properties -->
+    <gazebo reference="${link_prefix}base_footprint">
+      <kp>1e6</kp>
+      <kd>1.0</kd>
+      <mu1>0.3</mu1>
+      <mu2>0.3</mu2>
+      <minDepth>0.003</minDepth>
+    </gazebo>
+    <gazebo reference="${link_prefix}base_link">
+      <kp>1e6</kp>
+      <kd>1.0</kd>
+      <mu1>0.3</mu1>
+      <mu2>0.3</mu2>
+      <minDepth>0.003</minDepth>
+    </gazebo>
     <!-- rocker ODE properties -->
     <gazebo reference="${link_prefix}rocker_L_link">
       <kp>1e6</kp>
       <kd>1.0</kd>
+      <mu1>0.3</mu1>
+      <mu2>0.3</mu2>
       <minDepth>0.003</minDepth>
     </gazebo>
@@ -215,4 +239,6 @@
       <kp>1e6</kp>
       <kd>1.0</kd>
+      <mu1>0.3</mu1>
+      <mu2>0.3</mu2>
       <minDepth>0.003</minDepth>
     </gazebo>
@@ -220,7 +246,7 @@
     <gazebo reference="${link_prefix}wheel_FL_link">
       <kp>1e6</kp>
-      <kd>1.0</kd>
+      <kd>100.0</kd>
       <mu1>3.0</mu1>
-      <mu2>0.5</mu2>
+      <mu2>1.0</mu2>
       <fdir1>1 0 0</fdir1>
       <minDepth>0.003</minDepth>
@@ -228,7 +254,7 @@
     <gazebo reference="${link_prefix}wheel_FR_link">
       <kp>1e6</kp>
-      <kd>1.0</kd>
+      <kd>100.0</kd>
       <mu1>3.0</mu1>
-      <mu2>0.5</mu2>
+      <mu2>1.0</mu2>
       <fdir1>1 0 0</fdir1>
       <minDepth>0.003</minDepth>
@@ -236,7 +262,7 @@
     <gazebo reference="${link_prefix}wheel_RL_link">
       <kp>1e6</kp>
-      <kd>1.0</kd>
+      <kd>100.0</kd>
       <mu1>3.0</mu1>
-      <mu2>0.5</mu2>
+      <mu2>1.0</mu2>
       <fdir1>1 0 0</fdir1>
       <minDepth>0.003</minDepth>
@@ -244,7 +270,7 @@
     <gazebo reference="${link_prefix}wheel_RR_link">
       <kp>1e6</kp>
-      <kd>1.0</kd>
+      <kd>100.0</kd>
       <mu1>3.0</mu1>
-      <mu2>0.5</mu2>
+      <mu2>1.0</mu2>
       <fdir1>1 0 0</fdir1>
       <minDepth>0.003</minDepth>
@@ -295,4 +321,17 @@
       </plugin>
     </gazebo>
+    <gazebo reference="${link_prefix}imu_frame">
+      <sensor type="imu" name="leo_imu_sensor">
+        <update_rate>100</update_rate>
+        <plugin filename="libgazebo_ros_imu_sensor.so" name="imu_plugin">
+          <robotNamespace>${robot_ns}</robotNamespace>
+          <topicName>imu/data_raw</topicName>
+          <frameName>${link_prefix}imu_frame</frameName>
+          <updateRateHZ>100.0</updateRateHZ>
+          <gaussianNoise>0.01</gaussianNoise>
+          <initialOrientationAsReference>false</initialOrientationAsReference>
+        </plugin>
+      </sensor>
+    </gazebo>
     <ros2_control name="GazeboSystem" type="system">
       <hardware>

Commit message: Macros.xacro cleanup

File: leo_description/urdf/macros.xacro (robot description, xacro)
@@ -279,6 +279,6 @@
     <!-- camera -->
     <gazebo reference="${link_prefix}camera_frame">
-      <sensor name="camera" type="camera">
-          <camera name="leo_camera">
+      <sensor name="${link_prefix}camera" type="camera">
+          <camera name="${link_prefix}leo_camera">
               <horizontal_fov>1.9</horizontal_fov>
               <image>
@@ -308,5 +308,5 @@
           <update_rate>30</update_rate>
           <visualize>true</visualize>
-          <topic>camera/image_raw</topic>
+          <topic>${link_prefix}camera/image_raw</topic>
           <ignition_frame_id>${link_prefix}camera_frame</ignition_frame_id>
       </sensor>
@@ -325,85 +325,22 @@
         name="ignition::gazebo::systems::JointStatePublisher">
       </plugin>
-    <!--
-      <plugin
-        filename="ignition-gazebo-pose-publisher-system"
-        name="ignition::gazebo::systems::PosePublisher">
-        <publish_link_pose>true</publish_link_pose>
-        <use_pose_vector_msg>true</use_pose_vector_msg>
-        <static_publisher>true</static_publisher>
-        <static_update_frequency>1</static_update_frequency>
-      </plugin>-->
     </gazebo>
     <gazebo reference="${link_prefix}imu_frame">
-      <sensor type="imu" name="leo_imu_sensor">
+      <sensor type="imu" name="${link_prefix}leo_imu_sensor">
         <update_rate>100</update_rate>
         <visualize>true</visualize>
-        <topic>imu/data_raw</topic>
+        <topic>${link_prefix}imu/data_raw</topic>
         <always_on>1</always_on>
         <ignition_frame_id>${link_prefix}imu_frame</ignition_frame_id>
       </sensor>
     </gazebo>
-<!--
-    <ros2_control name="GazeboSystem" type="system">
-      <hardware>
-        <plugin>gazebo_ros2_control/GazeboSystem</plugin>
-      </hardware>
-      <joint name="rocker_L_joint">
-        <state_interface name="position"/>
-      </joint>
-      <joint name="rocker_R_joint">
-        <state_interface name="position"/>
-      </joint>
-      <joint name="wheel_FL_joint">
-        <command_interface name="velocity">
-          <param name="min">-6</param>
-          <param name="max">6</param>
-        </command_interface>
-        <state_interface name="position"/>
-        <state_interface name="velocity"/>
-        <state_interface name="effort"/>
-      </joint>
-      <joint name="wheel_RL_joint">
-        <command_interface name="velocity">
-          <param name="min">-6</param>
-          <param name="max">6</param>
-        </command_interface>
-        <state_interface name="position"/>
-        <state_interface name="velocity"/>
-        <state_interface name="effort"/>
-      </joint>
-      <joint name="wheel_FR_joint">
-        <command_interface name="velocity">
-          <param name="min">-6</param>
-          <param name="max">6</param>
-        </command_interface>
-        <state_interface name="position"/>
-        <state_interface name="velocity"/>
-        <state_interface name="effort"/>
-      </joint>
-      <joint name="wheel_RR_joint">
-        <command_interface name="velocity">
-          <param name="min">-6</param>
-          <param name="max">6</param>
-        </command_interface>
-        <state_interface name="position"/>
-        <state_interface name="velocity"/>
-        <state_interface name="effort"/>
-      </joint>
-    </ros2_control>
--->
     <gazebo>
-      <!--<plugin filename="libgazebo_ros2_control.so" name="gazebo_ros2_control">
-        <robot_param>robot_description</robot_param>
-        <robot_param_node>robot_state_publisher</robot_param_node>
-        <parameters>package://leo_description/config/controllers.yaml</parameters>
-      </plugin>-->
       <plugin
         filename="libignition-gazebo-diff-drive-system.so"
         name="ignition::gazebo::systems::DiffDrive">
-        <left_joint>wheel_FL_joint</left_joint>
-        <right_joint>wheel_FR_joint</right_joint>
-        <left_joint>wheel_RL_joint</left_joint>
-        <right_joint>wheel_RR_joint</right_joint>
+        <left_joint>${joint_prefix}wheel_FL_joint</left_joint>
+        <right_joint>${joint_prefix}wheel_FR_joint</right_joint>
+        <left_joint>${joint_prefix}wheel_RL_joint</left_joint>
+        <right_joint>${joint_prefix}wheel_RR_joint</right_joint>
         <wheel_separation>0.358</wheel_separation>
         <wheel_radius>0.0625</wheel_radius>
@@ -411,5 +348,7 @@
         <child_frame_id>${link_prefix}base_footprint</child_frame_id>
         <odom_publish_frequency>20</odom_publish_frequency>
-        <topic>cmd_vel</topic>
+        <topic>${link_prefix}cmd_vel</topic>
+        <odom_topic>${link_prefix}odom</odom_topic>
+        <tf_topic>${link_prefix}tf</tf_topic>
         <max_linear_acceleration>2.5</max_linear_acceleration>
         <max_angular_acceleration>3</max_angular_acceleration>
@@ -417,64 +356,5 @@
         <min_angular_acceleration>-3</min_angular_acceleration>
       </plugin>
-      <!--
-      <plugin filename="libignition-gazebo-mecanum-drive-system.so" name="ignition::gazebo::systems::MecanumDrive">
-        <front_left_joint>wheel_FL_joint</front_left_joint>
-        <front_right_joint>wheel_FR_joint</front_right_joint>
-        <back_left_joint>wheel_RL_joint</back_left_joint>
-        <back_right_joint>wheel_RR_joint</back_right_joint>
-        <wheel_separation>0.358</wheel_separation>
-        <wheel_radius>0.0625</wheel_radius>
-        <wheelbase>0.3</wheelbase>
-        <odom_publish_frequency>20</odom_publish_frequency>
-        <topic>cmd_vel</topic>
-        <frame_id>odom</frame_id>
-        <child_frame_id>${link_prefix}base_footprint</child_frame_id>
-      </plugin>      -->
-<!--
-       <plugin filename="libignition-gazebo-wheel-slip-system.so"
-          name="systems::WheelSlip">
-          <wheel link_name="wheel_FL_link">
-            <slip_compliance_lateral>0</slip_compliance_lateral>
-            <slip_compliance_longitudinal>0.1</slip_compliance_longitudinal>
-            <wheel_normal_force>100</wheel_normal_force>
-            <wheel_radius>0.0625</wheel_radius>
-          </wheel>
-          <wheel link_name="wheel_FR_link">
-            <slip_compliance_lateral>0</slip_compliance_lateral>
-            <slip_compliance_longitudinal>0.1</slip_compliance_longitudinal>
-            <wheel_normal_force>100</wheel_normal_force>
-            <wheel_radius>0.0625</wheel_radius>
-          </wheel>
-          <wheel link_name="wheel_RL_link">
-            <slip_compliance_lateral>0</slip_compliance_lateral>
-            <slip_compliance_longitudinal>0.1</slip_compliance_longitudinal>
-            <wheel_normal_force>80</wheel_normal_force>
-            <wheel_radius>0.0625</wheel_radius>
-          </wheel>
-          <wheel link_name="wheel_RR_link">
-            <slip_compliance_lateral>0</slip_compliance_lateral>
-            <slip_compliance_longitudinal>0.1</slip_compliance_longitudinal>
-            <wheel_normal_force>80</wheel_normal_force>
-            <wheel_radius>0.0625</wheel_radius>
-          </wheel>
-        </plugin>-->
-    </gazebo>
-<!--
-    <gazebo reference="${joint_prefix}base_joint">
-      <preserveFixedJoint>true</preserveFixedJoint>
-    </gazebo>
-    <gazebo reference="${joint_prefix}antenna_joint">
-      <preserveFixedJoint>true</preserveFixedJoint>
-    </gazebo>
-    <gazebo reference="${joint_prefix}camera_joint">
-      <preserveFixedJoint>true</preserveFixedJoint>
-    </gazebo>
-    <gazebo reference="${joint_prefix}camera_optical_joint">
-      <preserveFixedJoint>true</preserveFixedJoint>
-    </gazebo>
-    <gazebo reference="${joint_prefix}imu_joint">
-      <preserveFixedJoint>true</preserveFixedJoint>
-    </gazebo>
--->
+    </gazebo>
   </xacro:macro>
   <xacro:macro name="leo_sim"
@@ -483,11 +363,15 @@
                        robot_ns:=''">
     <xacro:property name="link_prefix" value=""/>
+    <xacro:property name="joint_prefix" value=""/>
     <xacro:if value="${robot_ns != '' and robot_ns != '/'}">
       <xacro:property name="link_prefix" value="${robot_ns}/"/>
+      <xacro:property name="joint_prefix" value="${robot_ns}/"/>
     </xacro:if>
     <xacro:leo default_antenna="${default_antenna}"
                rockers_fixed="false"
-               link_prefix="${link_prefix}"/>
-    <xacro:leo_gazebo robot_ns="${robot_ns}"/>
+               link_prefix="${link_prefix}"
+               joint_prefix="${joint_prefix}"/>
+    <xacro:leo_gazebo robot_ns="${robot_ns}"
+    joint_prefix="${joint_prefix}"/>
     <xacro:if value="${fixed}">
       <link name="world"/>
