Commit message: Fix gazebo launch warnings

File: leo_description/urdf/macros.xacro (robot description, xacro)
@@ -216,96 +216,144 @@
     <!-- base ODE properties -->
     <gazebo reference="${link_prefix}base_footprint">
-      <kp>1e6</kp>
-      <kd>1.0</kd>
-      <mu>0.3</mu>
-      <mu2>0.3</mu2>
-      <minDepth>0.003</minDepth>
+      <collision>
+        <surface>
+          <friction>
+            <ode>
+              <mu>0.3</mu>
+              <mu2>0.3</mu2>
+            </ode>
+            <bullet>
+              <friction>1</friction>
+              <friction2>1</friction2>
+              <rolling_friction>0.1</rolling_friction>
+            </bullet>
+          </friction>
+        </surface>
+      </collision>
     </gazebo>
     <gazebo reference="${link_prefix}base_link">
-      <kp>1e6</kp>
-      <kd>1.0</kd>
-      <mu>0.3</mu>
-      <mu2>0.3</mu2>
-      <minDepth>0.003</minDepth>
+      <collision>
+        <surface>
+          <friction>
+            <ode>
+              <mu>0.3</mu>
+              <mu2>0.3</mu2>
+            </ode>
+            <bullet>
+              <friction>1</friction>
+              <friction2>1</friction2>
+              <rolling_friction>0.1</rolling_friction>
+            </bullet>
+          </friction>
+        </surface>
+      </collision>
     </gazebo>
     <!-- rocker ODE properties -->
     <gazebo reference="${link_prefix}rocker_L_link">
-      <kp>1e6</kp>
-      <kd>1.0</kd>
-      <mu>0.3</mu>
-      <mu2>0.3</mu2>
-      <minDepth>0.003</minDepth>
+      <collision>
+        <surface>
+          <friction>
+            <ode>
+              <mu>0.3</mu>
+              <mu2>0.3</mu2>
+            </ode>
+            <bullet>
+              <friction>1</friction>
+              <friction2>1</friction2>
+              <rolling_friction>0.1</rolling_friction>
+            </bullet>
+          </friction>
+        </surface>
+      </collision>
     </gazebo>
     <gazebo reference="${link_prefix}rocker_R_link">
-      <kp>1e6</kp>
-      <kd>1.0</kd>
-      <mu>0.3</mu>
-      <mu2>0.3</mu2>
-      <minDepth>0.003</minDepth>
+      <collision>
+        <surface>
+          <friction>
+            <ode>
+              <mu>0.3</mu>
+              <mu2>0.3</mu2>
+            </ode>
+            <bullet>
+              <friction>1</friction>
+              <friction2>1</friction2>
+              <rolling_friction>0.1</rolling_friction>
+            </bullet>
+          </friction>
+        </surface>
+      </collision>
     </gazebo>
     <!-- wheel ODE properties -->
     <gazebo reference="${link_prefix}wheel_FL_link">
-      <surface>
-        <friction>
-          <ode>
-            <mu>3.0</mu>
-            <mu2>1.0</mu2>
-            <fdir1>1 0 0</fdir1>
-          </ode>
-          <bullet>
-            <friction>1</friction>
-            <friction2>1</friction2>
-            <rolling_friction>0.1</rolling_friction>
-          </bullet>
-        </friction>
-      </surface>
+      <collision>
+        <surface>
+          <friction>
+            <ode>
+              <mu>1.0</mu>
+              <mu2>1.0</mu2>
+              <fdir1>0 0 0</fdir1>
+            </ode>
+            <bullet>
+              <friction>1</friction>
+              <friction2>1</friction2>
+              <rolling_friction>0.1</rolling_friction>
+            </bullet>
+          </friction>
+        </surface>
+      </collision>
     </gazebo>
     <gazebo reference="${link_prefix}wheel_FR_link">
-      <surface>
-        <friction>
-          <ode>
-            <mu>3.0</mu>
-            <mu2>1.0</mu2>
-            <fdir1>1 0 0</fdir1>
-          </ode>
-          <bullet>
-            <friction>1</friction>
-            <friction2>1</friction2>
-            <rolling_friction>0.1</rolling_friction>
-          </bullet>
-        </friction>
-      </surface>
+      <collision>
+        <surface>
+          <friction>
+            <ode>
+              <mu>1.0</mu>
+              <mu2>1.0</mu2>
+              <fdir1>0 0 0</fdir1>
+            </ode>
+            <bullet>
+              <friction>1</friction>
+              <friction2>1</friction2>
+              <rolling_friction>0.1</rolling_friction>
+            </bullet>
+          </friction>
+        </surface>
+      </collision>
     </gazebo>
     <gazebo reference="${link_prefix}wheel_RL_link">
-      <surface>
-        <friction>
-          <ode>
-            <mu>3.0</mu>
-            <mu2>1.0</mu2>
-            <fdir1>1 0 0</fdir1>
-          </ode>
-          <bullet>
-            <friction>1</friction>
-            <friction2>1</friction2>
-            <rolling_friction>0.1</rolling_friction>
-          </bullet>
-        </friction>
-      </surface>
+      <collision>
+        <surface>
+          <friction>
+            <ode>
+              <mu>1.0</mu>
+              <mu2>1.0</mu2>
+              <fdir1>0 0 0</fdir1>
+            </ode>
+            <bullet>
+              <friction>1</friction>
+              <friction2>1</friction2>
+              <rolling_friction>0.1</rolling_friction>
+            </bullet>
+          </friction>
+        </surface>
+      </collision>
     </gazebo>
     <gazebo reference="${link_prefix}wheel_RR_link">
-      <surface>
-        <friction>
-          <ode>
-            <mu>3.0</mu>
-            <mu2>1.0</mu2>
-            <fdir1>1 0 0</fdir1>
-          </ode>
-          <bullet>
-            <friction>1</friction>
-            <friction2>1</friction2>
-            <rolling_friction>0.1</rolling_friction>
-          </bullet>
-        </friction>
-      </surface>
+      <collision>
+        <surface>
+          <friction>
+            <ode>
+              <mu>1.0</mu>
+              <mu2>1.0</mu2>
+              <fdir1>0 0 0</fdir1>
+            </ode>
+            <bullet>
+              <friction>1</friction>
+              <friction2>1</friction2>
+              <rolling_friction>0.1</rolling_friction>
+            </bullet>
+          </friction>
+        </surface>
+      </collision>
     </gazebo>
     <!-- camera -->

Commit message: Remove joint prefix

File: leo_description/urdf/macros.xacro (robot description, xacro)
@@ -6,5 +6,4 @@
                        footprint_link:=true
                        link_prefix:=''
-                       joint_prefix:=''
                        imu_translation:='0.0628 -0.0314 -0.0393'">
     <xacro:macro name="rocker_link" params="name">
@@ -122,5 +121,5 @@
     <!-- JOINTS -->
     <xacro:if value="${footprint_link}">
-      <joint name="${joint_prefix}base_joint" type="fixed">
+      <joint name="base_joint" type="fixed">
         <origin xyz="0 0 0.19783" rpy="0 0 0"/>
         <parent link="${link_prefix}base_footprint"/>
@@ -134,5 +133,5 @@
       <xacro:property name="rockers_joint_type" value="revolute"/>
     </xacro:unless>
-    <joint name="${joint_prefix}rocker_L_joint" type="${rockers_joint_type}">
+    <joint name="rocker_L_joint" type="${rockers_joint_type}">
       <origin xyz="0.00263 0.14167 -0.04731" rpy="0 0 ${pi}"/>
       <parent link="${link_prefix}base_link"/>
@@ -142,5 +141,5 @@
       <dynamics friction="1.0" damping="0.1"/>
     </joint>
-    <joint name="${joint_prefix}rocker_R_joint" type="${rockers_joint_type}">
+    <joint name="rocker_R_joint" type="${rockers_joint_type}">
       <origin xyz="0.00263 -0.14167 -0.04731" rpy="0 0 0"/>
       <parent link="${link_prefix}base_link"/>
@@ -151,5 +150,5 @@
       <mimic joint="rocker_L_joint"/>
     </joint>
-    <joint name="${joint_prefix}wheel_FL_joint" type="continuous">
+    <joint name="wheel_FL_joint" type="continuous">
       <origin xyz="-0.15256 -0.08214 -0.08802" rpy="0 0 0"/>
       <parent link="${link_prefix}rocker_L_link"/>
@@ -159,5 +158,5 @@
       <dynamics friction="0.3125" damping="0.1"/>
     </joint>
-    <joint name="${joint_prefix}wheel_RL_joint" type="continuous">
+    <joint name="wheel_RL_joint" type="continuous">
       <origin xyz="0.15256 -0.08214 -0.08802" rpy="0 0 0"/>
       <parent link="${link_prefix}rocker_L_link"/>
@@ -167,5 +166,5 @@
       <dynamics friction="0.3125" damping="0.1"/>
     </joint>
-    <joint name="${joint_prefix}wheel_FR_joint" type="continuous">
+    <joint name="wheel_FR_joint" type="continuous">
       <origin xyz="0.15256 -0.08214 -0.08802" rpy="0 0 0"/>
       <parent link="${link_prefix}rocker_R_link"/>
@@ -175,5 +174,5 @@
       <dynamics friction="0.3125" damping="0.1"/>
     </joint>
-    <joint name="${joint_prefix}wheel_RR_joint" type="continuous">
+    <joint name="wheel_RR_joint" type="continuous">
       <origin xyz="-0.15256 -0.08214 -0.08802" rpy="0 0 0"/>
       <parent link="${link_prefix}rocker_R_link"/>
@@ -184,5 +183,5 @@
     </joint>
     <xacro:if value="${default_antenna}">
-      <joint name="${joint_prefix}antenna_joint" type="fixed">
+      <joint name="antenna_joint" type="fixed">
         <origin xyz="-0.0052 0.056 -0.0065" rpy="0 0 0"/>
         <parent link="${link_prefix}base_link"/>
@@ -190,15 +189,15 @@
       </joint>
     </xacro:if>
-    <joint name="${joint_prefix}camera_joint" type="fixed">
+    <joint name="camera_joint" type="fixed">
       <origin xyz="0.0971 0 -0.0427" rpy="0 0.2094 0"/>
       <parent link="${link_prefix}base_link"/>
       <child link="${link_prefix}camera_frame"/>
     </joint>
-    <joint name="${joint_prefix}camera_optical_joint" type="fixed">
+    <joint name="camera_optical_joint" type="fixed">
       <origin xyz="0 0 0" rpy="-${pi/2} 0.0 -${pi/2}"/>
       <parent link="${link_prefix}camera_frame"/>
       <child link="${link_prefix}camera_optical_frame"/>
     </joint>
-    <joint name="${joint_prefix}imu_joint" type="fixed">
+    <joint name="imu_joint" type="fixed">
       <origin xyz="${imu_translation}" rpy="0 0 0"/>
       <parent link="${link_prefix}base_link"/>
@@ -420,8 +419,8 @@
         filename="libignition-gazebo-diff-drive-system.so"
         name="ignition::gazebo::systems::DiffDrive">
-        <left_joint>${joint_prefix}wheel_FL_joint</left_joint>
-        <right_joint>${joint_prefix}wheel_FR_joint</right_joint>
-        <left_joint>${joint_prefix}wheel_RL_joint</left_joint>
-        <right_joint>${joint_prefix}wheel_RR_joint</right_joint>
+        <left_joint>wheel_FL_joint</left_joint>
+        <right_joint>wheel_FR_joint</right_joint>
+        <left_joint>wheel_RL_joint</left_joint>
+        <right_joint>wheel_RR_joint</right_joint>
         <wheel_separation>0.358</wheel_separation>
         <wheel_radius>0.0625</wheel_radius>
@@ -451,8 +450,6 @@
     <xacro:leo default_antenna="${default_antenna}"
                rockers_fixed="false"
-               link_prefix="${link_prefix}"
-               joint_prefix="${joint_prefix}"/>
-    <xacro:leo_gazebo robot_ns="${robot_ns}"
-    joint_prefix="${joint_prefix}"/>
+               link_prefix="${link_prefix}"/>
+    <xacro:leo_gazebo robot_ns="${robot_ns}"/>
     <xacro:if value="${fixed}">
       <link name="world"/>

Commit message: Add joints prefix param to all joints

File: leo_description/urdf/macros.xacro (robot description, xacro)
@@ -122,5 +122,5 @@
     <!-- JOINTS -->
     <xacro:if value="${footprint_link}">
-      <joint name="base_joint" type="fixed">
+      <joint name="${joint_prefix}base_joint" type="fixed">
         <origin xyz="0 0 0.19783" rpy="0 0 0"/>
         <parent link="${link_prefix}base_footprint"/>
@@ -134,5 +134,5 @@
       <xacro:property name="rockers_joint_type" value="revolute"/>
     </xacro:unless>
-    <joint name="rocker_L_joint" type="${rockers_joint_type}">
+    <joint name="${joint_prefix}rocker_L_joint" type="${rockers_joint_type}">
       <origin xyz="0.00263 0.14167 -0.04731" rpy="0 0 ${pi}"/>
       <parent link="${link_prefix}base_link"/>
@@ -142,5 +142,5 @@
       <dynamics friction="1.0" damping="0.1"/>
     </joint>
-    <joint name="rocker_R_joint" type="${rockers_joint_type}">
+    <joint name="${joint_prefix}rocker_R_joint" type="${rockers_joint_type}">
       <origin xyz="0.00263 -0.14167 -0.04731" rpy="0 0 0"/>
       <parent link="${link_prefix}base_link"/>
@@ -151,5 +151,5 @@
       <mimic joint="rocker_L_joint"/>
     </joint>
-    <joint name="wheel_FL_joint" type="continuous">
+    <joint name="${joint_prefix}wheel_FL_joint" type="continuous">
       <origin xyz="-0.15256 -0.08214 -0.08802" rpy="0 0 0"/>
       <parent link="${link_prefix}rocker_L_link"/>
@@ -159,5 +159,5 @@
       <dynamics friction="0.3125" damping="0.1"/>
     </joint>
-    <joint name="wheel_RL_joint" type="continuous">
+    <joint name="${joint_prefix}wheel_RL_joint" type="continuous">
       <origin xyz="0.15256 -0.08214 -0.08802" rpy="0 0 0"/>
       <parent link="${link_prefix}rocker_L_link"/>
@@ -167,5 +167,5 @@
       <dynamics friction="0.3125" damping="0.1"/>
     </joint>
-    <joint name="wheel_FR_joint" type="continuous">
+    <joint name="${joint_prefix}wheel_FR_joint" type="continuous">
       <origin xyz="0.15256 -0.08214 -0.08802" rpy="0 0 0"/>
       <parent link="${link_prefix}rocker_R_link"/>
@@ -175,5 +175,5 @@
       <dynamics friction="0.3125" damping="0.1"/>
     </joint>
-    <joint name="wheel_RR_joint" type="continuous">
+    <joint name="${joint_prefix}wheel_RR_joint" type="continuous">
       <origin xyz="-0.15256 -0.08214 -0.08802" rpy="0 0 0"/>
       <parent link="${link_prefix}rocker_R_link"/>
@@ -184,5 +184,5 @@
     </joint>
     <xacro:if value="${default_antenna}">
-      <joint name="antenna_joint" type="fixed">
+      <joint name="${joint_prefix}antenna_joint" type="fixed">
         <origin xyz="-0.0052 0.056 -0.0065" rpy="0 0 0"/>
         <parent link="${link_prefix}base_link"/>
@@ -190,15 +190,15 @@
       </joint>
     </xacro:if>
-    <joint name="camera_joint" type="fixed">
+    <joint name="${joint_prefix}camera_joint" type="fixed">
       <origin xyz="0.0971 0 -0.0427" rpy="0 0.2094 0"/>
       <parent link="${link_prefix}base_link"/>
       <child link="${link_prefix}camera_frame"/>
     </joint>
-    <joint name="camera_optical_joint" type="fixed">
+    <joint name="${joint_prefix}camera_optical_joint" type="fixed">
       <origin xyz="0 0 0" rpy="-${pi/2} 0.0 -${pi/2}"/>
       <parent link="${link_prefix}camera_frame"/>
       <child link="${link_prefix}camera_optical_frame"/>
     </joint>
-    <joint name="imu_joint" type="fixed">
+    <joint name="${joint_prefix}imu_joint" type="fixed">
       <origin xyz="${imu_translation}" rpy="0 0 0"/>
       <parent link="${link_prefix}base_link"/>
@@ -208,6 +208,5 @@
   <!-- LEO GAZEBO -->
   <xacro:macro name="leo_gazebo"
-               params="robot_ns:=''
-               joint_prefix:=''">
+               params="robot_ns:='''">
     <xacro:property name="link_prefix" value=""/>
     <xacro:if value="${robot_ns != '' and robot_ns != '/'}">
@@ -447,8 +446,6 @@
                        robot_ns:=''">
     <xacro:property name="link_prefix" value=""/>
-    <xacro:property name="joint_prefix" value=""/>
     <xacro:if value="${robot_ns != '' and robot_ns != '/'}">
       <xacro:property name="link_prefix" value="${robot_ns}/"/>
-      <xacro:property name="joint_prefix" value="${robot_ns}/"/>
     </xacro:if>
     <xacro:leo default_antenna="${default_antenna}"
